File: PeakHoldPWMDriver_V0.3.2/PeakHoldPWMDriver.kicad_pcb (KiCad board)
At the start: 2 copper layers, 100.1 x 50 mm, 122 parts, among them J1 RND 205-00203, J2 RND 205-00205, Q1 2N7002, Q10 2N7002, Q11 2N7002, Q12 2N7002, Q13 TSM2309, Q14 IRLL 024N, Q15 TSM2309, Q16 IRLL 024N, Q17 TSM2309, Q18 TSM2309, Q19 TSM2309, Q2 2N7002, Q20 TSM2309, Q3 2N7002, Q4 2N7002, Q5 TSM2309, Q6 TSM2309, Q7 IRLL 024N, Q8 IRLL 024N, Q9 2N7002, U1 74HC32, U2 LM2901, U3 74HC74, U4 LTC6992, U5 74HC74, U6 LM340, U7 74HC08, U8 74HC08

Commit message: Added position csv and BOM files in JLCPCB placement list format
Parts:
- D3: value BAV103 -> LL4148
- R6: value 180R -> 470R
Changed lines of the file:
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@@
     (visible_elements FFFFFF7F)
     (pcbplotparams
-      (layerselection 0x010fc_ffffffff)
+      (layerselection 0x010f0_ffffffff)
       (usegerberextensions false)
       (usegerberattributes false)
@@
       (psa4output false)
       (plotreference true)
-      (plotvalue true)
+      (plotvalue false)
       (plotinvisibletext false)
-      (padsonsilk false)
+      (padsonsilk true)
       (subtractmaskfromsilk false)
       (outputformat 1)
@@
       (effects (font (size 1 1) (thickness 0.15)))
     )
-    (fp_text user %R (at 0 0) (layer F.Fab)
-      (effects (font (size 0.4 0.4) (thickness 0.06)))
-    )
     (fp_line (start -0.8 0.4) (end -0.8 -0.4) (layer F.Fab) (width 0.1))
     (fp_line (start -0.8 -0.4) (end 0.8 -0.4) (layer F.Fab) (width 0.1))
@@
     (fp_line (start 1.65 -0.73) (end 1.65 0.73) (layer F.CrtYd) (width 0.05))
     (fp_line (start 1.65 0.73) (end -1.65 0.73) (layer F.CrtYd) (width 0.05))
+    (fp_text user %R (at 0 0) (layer F.Fab)
+      (effects (font (size 0.4 0.4) (thickness 0.06)))
+    )
     (pad 2 smd roundrect (at 0.875 0 180) (size 1.05 0.95) (layers F.Cu F.Paste F.Mask) (roundrect_rratio 0.25)
       (net 10 VREF))
@@
       (effects (font (size 1 1) (thickness 0.15)))
     )
-    (fp_text user %R (at 0 0) (layer F.Fab)
-      (effects (font (size 0.4 0.4) (thickness 0.06)))
-    )
     (fp_line (start -0.8 0.4) (end -0.8 -0.4) (layer F.Fab) (width 0.1))
     (fp_line (start -0.8 -0.4) (end 0.8 -0.4) (layer F.Fab) (width 0.1))
@@
     (fp_line (start 1.65 -0.73) (end 1.65 0.73) (layer F.CrtYd) (width 0.05))
     (fp_line (start 1.65 0.73) (end -1.65 0.73) (layer F.CrtYd) (width 0.05))
+    (fp_text user %R (at 0 0) (layer F.Fab)
+      (effects (font (size 0.4 0.4) (thickness 0.06)))
+    )
     (pad 2 smd roundrect (at 0.875 0 180) (size 1.05 0.95) (layers F.Cu F.Paste F.Mask) (roundrect_rratio 0.25)
       (net 1 5V))
@@
       (effects (font (size 1 1) (thickness 0.15)))
     )
-    (fp_text user %R (at 0 0) (layer F.Fab)
-      (effects (font (size 0.4 0.4) (thickness 0.06)))
-    )
     (fp_line (start -0.8 0.4) (end -0.8 -0.4) (layer F.Fab) (width 0.1))
     (fp_line (start -0.8 -0.4) (end 0.8 -0.4) (layer F.Fab) (width 0.1))
@@
     (fp_line (start 1.65 -0.73) (end 1.65 0.73) (layer F.CrtYd) (width 0.05))
     (fp_line (start 1.65 0.73) (end -1.65 0.73) (layer F.CrtYd) (width 0.05))
+    (fp_text user %R (at 0 0) (layer F.Fab)
+      (effects (font (size 0.4 0.4) (thickness 0.06)))
+    )
     (pad 2 smd roundrect (at 0.875 0) (size 1.05 0.95) (layers F.Cu F.Paste F.Mask) (roundrect_rratio 0.25)
       (net 1 5V))
@@
       (effects (font (size 1 1) (thickness 0.15)))
     )
-    (fp_text user %R (at 0 0 90) (layer F.Fab)
-      (effects (font (size 0.4 0.4) (thickness 0.06)))
-    )
     (fp_line (start -0.8 0.4) (end -0.8 -0.4) (layer F.Fab) (width 0.1))
     (fp_line (start -0.8 -0.4) (end 0.8 -0.4) (layer F.Fab) (width 0.1))
@@
     (fp_line (start 1.65 -0.73) (end 1.65 0.73) (layer F.CrtYd) (width 0.05))
     (fp_line (start 1.65 0.73) (end -1.65 0.73) (layer F.CrtYd) (width 0.05))
+    (fp_text user %R (at 0 0 90) (layer F.Fab)
+      (effects (font (size 0.4 0.4) (thickness 0.06)))
+    )
     (pad 2 smd roundrect (at 0.875 0 90) (size 1.05 0.95) (layers F.Cu F.Paste F.Mask) (roundrect_rratio 0.25)
       (net 1 5V))
@@
       (effects (font (size 1 1) (thickness 0.15)))
     )
-    (fp_text user %R (at 0 0 90) (layer F.Fab)
-      (effects (font (size 0.4 0.4) (thickness 0.06)))
-    )
     (fp_line (start -0.8 0.4) (end -0.8 -0.4) (layer F.Fab) (width 0.1))
     (fp_line (start -0.8 -0.4) (end 0.8 -0.4) (layer F.Fab) (width 0.1))
@@
     (fp_line (start 1.65 -0.73) (end 1.65 0.73) (layer F.CrtYd) (width 0.05))
     (fp_line (start 1.65 0.73) (end -1.65 0.73) (layer F.CrtYd) (width 0.05))
+    (fp_text user %R (at 0 0 90) (layer F.Fab)
+      (effects (font (size 0.4 0.4) (thickness 0.06)))
+    )
     (pad 2 smd roundrect (at 0.875 0 90) (size 1.05 0.95) (layers F.Cu F.Paste F.Mask) (roundrect_rratio 0.25)
       (net 1 5V))
@@
       (effects (font (size 1 1) (thickness 0.15)))
     )
-    (fp_text user %R (at 0 0) (layer F.Fab)
-      (effects (font (size 0.4 0.4) (thickness 0.06)))
-    )
     (fp_line (start -0.8 0.4) (end -0.8 -0.4) (layer F.Fab) (width 0.1))
     (fp_line (start -0.8 -0.4) (end 0.8 -0.4) (layer F.Fab) (width 0.1))
@@
     (fp_line (start 1.65 -0.73) (end 1.65 0.73) (layer F.CrtYd) (width 0.05))
     (fp_line (start 1.65 0.73) (end -1.65 0.73) (layer F.CrtYd) (width 0.05))
+    (fp_text user %R (at 0 0) (layer F.Fab)
+      (effects (font (size 0.4 0.4) (thickness 0.06)))
+    )
     (pad 2 smd roundrect (at 0.875 0) (size 1.05 0.95) (layers F.Cu F.Paste F.Mask) (roundrect_rratio 0.25)
       (net 1 5V))
@@
       (effects (font (size 1 1) (thickness 0.15)))
     )
-    (fp_text value BAV103 (at 0 1.75) (layer F.Fab)
+    (fp_text value LL4148 (at 0 1.75) (layer F.Fab)
       (effects (font (size 1 1) (thickness 0.15)))
     )
@@
       (effects (font (size 1 1) (thickness 0.15)))
     )
-    (fp_text value 180R (at 0 1.43) (layer F.Fab)
+    (fp_text value 470R (at 0 1.43) (layer F.Fab)
       (effects (font (size 1 1) (thickness 0.15)))
     )
@@
   (segment (start 183.674285 67.346999) (end 179.229999 67.346999) (width 0.25) (layer B.Cu) (net 10))
   (segment (start 174.498 87.064998) (end 174.280999 87.281999) (width 0.25) (layer B.Cu) (net 10))
+  (segment (start 172.974 82.55) (end 173.030979 82.493021) (width 0.25) (layer F.Cu) (net 10))
+  (segment (start 173.030979 82.493021) (end 173.284979 82.493021) (width 0.25) (layer F.Cu) (net 10))
+  (via (at 173.482 82.804) (size 0.8) (drill 0.4) (layers F.Cu B.Cu) (net 10))
+  (segment (start 173.369 82.804) (end 173.482 82.804) (width 0.25) (layer F.Cu) (net 10))
+  (segment (start 173.953001 82.332999) (end 174.280999 82.332999) (width 0.25) (layer B.Cu) (net 10))
+  (segment (start 173.482 82.804) (end 173.953001 82.332999) (width 0.25) (layer B.Cu) (net 10))
   (via (at 161.253 105.664) (size 0.8) (drill 0.4) (layers F.Cu B.Cu) (net 11))
   (segment (start 157.5735 105.664) (end 161.253 105.664) (width 0.25) (layer F.Cu) (net 11) (status 10))
@@
   (segment (start 155.277822 76.454) (end 157.008999 78.185177) (width 0.25) (layer F.Cu) (net 33))
   (segment (start 143.002 76.454) (end 155.277822 76.454) (width 0.25) (layer F.Cu) (net 33))
-  (segment (start 172.974 82.55) (end 173.030979 82.493021) (width 0.25) (layer F.Cu) (net 10))
-  (segment (start 173.030979 82.493021) (end 173.284979 82.493021) (width 0.25) (layer F.Cu) (net 10))
-  (via (at 173.482 82.804) (size 0.8) (drill 0.4) (layers F.Cu B.Cu) (net 10))
-  (segment (start 173.369 82.804) (end 173.482 82.804) (width 0.25) (layer F.Cu) (net 10))
-  (segment (start 173.953001 82.332999) (end 174.280999 82.332999) (width 0.25) (layer B.Cu) (net 10))
-  (segment (start 173.482 82.804) (end 173.953001 82.332999) (width 0.25) (layer B.Cu) (net 10))
   (via (at 177.375369 78.121303) (size 0.8) (drill 0.4) (layers F.Cu B.Cu) (net 33))
   (segment (start 177.375369 80.651631) (end 177.375369 78.121303) (width 0.25) (layer B.Cu) (net 33))
